Commit message: adding the tracker and follower package

File: description/camera.xacro (robot description, xacro)
@@ -4,5 +4,5 @@
         <parent link="chassis"/>
         <child link="camera_link"/>
-        <origin xyz="0.305 0 0.08" rpy="0 0 0"/>
+        <origin xyz="0.305 0 0.08" rpy="0 0.18 0"/>
     </joint>
     <link name="camera_link">

File: description/robot.urdf.xacro (robot description, xacro)
@@ -5,5 +5,5 @@
     <!-- <xacro:include filename="ros2_control.xacro" /> -->
     <xacro:include filename="lidar.xacro" />
-    <xacro:include filename="depth_camera.xacro" />
-    <!--<xacro:include filename="camera.xacro" />-->
+    <xacro:include filename="camera.xacro" />
+    <!--<xacro:include filename="depth_camera.xacro" />-->
 </robot>
